File: PowerMonitor.kicad_pcb (KiCad board)
At the start: 2 copper layers, 100 x 95 mm, 84 parts, among them J1 Conn_01x01, J10 TEST_1P, J11 TEST_1P, J12 TEST_1P, J13 TEST_1P, J14 TEST_1P, J15 TEST_1P, J16 Conn_01x03, J2 Conn_01x01, J3 Conn_01x01, J4 Conn_01x01, J5 Conn_01x01, J6 Conn_01x01, J7 Conn_01x01, J8 Conn_01x10, J9 TEST_1P, K1 T9AS5D12-5, K2 KEMET_UA2_5NJ, P1 Keystone_4912, P2 Keystone_4912, P3 Keystone_4912, P4 Keystone_4912, Q1 DMN3067LW, Q2 DMN3067LW, Q3 DMN3067LW, U1 IRM-02-5S, U2 IRM-05-5, U3 MCP39F521, U4 LP5907MFX-3.3, U5 ISO7731FDBQ, U6 ISO1540D

Commit message: placwmwnt v0.2
Parts:
- added REF**: MountingHole_3.2mm_M3, Mounting_Holes:MountingHole_3.2mm_M3, F.Cu at (196.4, 53.4)
- added REF**: MountingHole_3.2mm_M3, Mounting_Holes:MountingHole_3.2mm_M3, F.Cu at (196.6, 111.6)
- added REF**: MountingHole_3.2mm_M3, Mounting_Holes:MountingHole_3.2mm_M3, F.Cu at (196.4, 23.4)
- added REF**: MountingHole_3.2mm_M3, Mounting_Holes:MountingHole_3.2mm_M3, F.Cu at (103.4, 111.6)
- added REF**: MountingHole_3.2mm_M3, Mounting_Holes:MountingHole_3.2mm_M3, F.Cu at (103.8, 53.8)
- added REF**: MountingHole_3.2mm_M3, Mounting_Holes:MountingHole_3.2mm_M3, F.Cu at (103.2, 23.2)
- D1, D2, K2: moved to B.Cu
- moved P4 108.5 mm to (108.0, 43.0), turned to 270 degrees
- moved C4 106.0 mm to (174.8, 40.8), turned to 180 degrees
- moved R19 105.0 mm to (162.8, 72.0)
- moved P2 97.1 mm to (108.0, 31.4), turned to 270 degrees
- moved J8 95.5 mm to (167.2, 113.0), turned to 90 degrees
- moved D4 94.8 mm to (178.8, 22.0), turned to 180 degrees
- moved Q2 94.6 mm to (161.6, 23.6)
- moved D3 90.8 mm to (171.8, 22.0)
- moved C8 90.2 mm to (159.2, 64.8), turned to 270 degrees
- moved C7 89.5 mm to (168.2, 65.0), turned to 270 degrees
- moved R20 88.4 mm to (196.8, 72.6), turned to 270 degrees
- moved C3 79.4 mm to (179.6, 40.8), turned to 180 degrees
- moved R5 78.0 mm to (162.2, 42.0), turned to 270 degrees
- moved C2 71.5 mm to (165.6, 47.4), turned to 270 degrees
- moved L1 69.8 mm to (157.6, 43.2), turned to 0 degrees
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Connections:
- D1 pad 2: +5V -> Net-(D1-Pad2)
- D2 pad 1: Net-(D1-Pad1) -> +5V
- D2 pad 2: Net-(D2-Pad2) -> Net-(D1-Pad2)
- F1 pad 1: Net-(F1-Pad1) -> /Line_fused
- K1 pad 1: Net-(D2-Pad2) -> Net-(D1-Pad1)
- L2 pad 2: /Line_In -> /Line_fused
- L3 pad 2: Net-(K2-Pad6) -> Net-(K2-Pad3)
- L4 pad 2: Net-(K2-Pad3) -> Net-(K2-Pad6)
- Q1 pad 3: Net-(D2-Pad2) -> Net-(D1-Pad1)
- RV1 pad 1: Net-(F1-Pad1) -> /Line_fused
- U1 pad 1: Net-(F1-Pad1) -> /Line_fused
- U2 pad 1: Net-(F1-Pad1) -> /Line_fused

Commit message: layout started
Parts:
- added C15: 2.2uF 25V, Capacitors_SMD:C_0805, F.Cu at (173.8, 107.8)
- added J17: TEST_1P, nightmechanic_pcb:Keystone_50XX_TP, F.Cu at (165.0, 84.2)
- L1: moved to B.Cu
- moved J10 99.6 mm to (160.8, 51.8)
- moved J12 99.0 mm to (159.6, 112.0)
- moved J11 92.8 mm to (164.4, 72.8)
- moved J5 84.6 mm to (165.4, 51.2)
- moved J15 83.4 mm to (190.4, 100.2)
- moved J9 77.7 mm to (184.0, 49.6)
- moved J2 76.1 mm to (167.4, 51.2)
- moved J1 74.0 mm to (165.4, 53.2)
- moved J13 73.8 mm to (190.2, 107.2)
- moved J6 73.8 mm to (174.6, 61.2)
- moved J14 72.4 mm to (196.8, 82.8)
- moved J4 66.0 mm to (178.6, 61.2)
- moved J3 65.0 mm to (176.6, 61.2)
- moved J7 58.2 mm to (188.4, 73.2)
- moved J16 46.6 mm to (177.4, 103.0), turned to 90 degrees
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Connections:
- L2 pad 1: Net-(L2-Pad1) -> Net-(C1-Pad1)
- L2 pad 2: /Line_fused -> Net-(L2-Pad2)
- R1 pad 2: Net-(L2-Pad1) -> /Line_fused
- R4 pad 1: Net-(C1-Pad1) -> Net-(L2-Pad2)
Routing:
- net +5V: track 0.00 -> 164.1 mm, vias 0 -> 1
- net GNDD: track 0.00 -> 137.3 mm, vias 0 -> 34
- net +3V3: track 0.00 -> 116.1 mm, vias 0 -> 2
- net +3.3V_ISO: track 0.00 -> 95.6 mm, vias 0 -> 2
- net +5V_ISO: track 0.00 -> 73.9 mm
- net /Line_fused: track 0.00 -> 70.2 mm
- net +3.3VA: track 0.00 -> 58.2 mm, vias 0 -> 1
- net GNDA: track 0.00 -> 33.2 mm, vias 0 -> 16
- net /Line_In: track 0.00 -> 32.1 mm
- net GND: track 0.00 -> 29.7 mm, vias 0 -> 10
- net /SW_CTRL_ISO: track 0.00 -> 23.2 mm
- net /MCLR_ISO: track 0.00 -> 22.4 mm
- net /EVENT_ISO: track 0.00 -> 21.6 mm
- net /SCL_ISO: track 0.00 -> 21.5 mm
- net /SDA_ISO: track 0.00 -> 21.3 mm
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- added copper zone on F.Cu, net /Line_fused
- added copper zone on B.Cu, net GND
- added copper zone on B.Cu, net GNDA
- added copper zone on B.Cu, net GNDD
- added copper zone on F.Cu, net GNDD
- added copper zone on B.Cu, net Net-(K1-Pad4)
- added copper zone on B.Cu, net Net-(K1-Pad5)
- added copper zone on B.Cu, net Net-(K2-Pad2)
- added copper zone on B.Cu, net Net-(K2-Pad4)
Other:
- outline, holes or cut-outs redrawn
- net class 0_4 added: clearance 0.19, trace_width 0.4, via_dia 0.6, via_drill 0.4
- net class 0_5 added: clearance 0.19, trace_width 0.5, via_dia 0.6, via_drill 0.4
- net class 3V_ISO added: clearance 0.19, trace_width 0.6, via_dia 0.6, via_drill 0.4
- net class 5V_ISO added: clearance 0.19, trace_width 1.5, via_dia 1, via_drill 0.5
- net class AC_L added: clearance 0.19, trace_width 2.5, via_dia 0.6, via_drill 0.4
- net class Default: clearance 0.2 -> 0.19; trace_width 0.25 -> 0.28
- net class GND_ISO added: clearance 0.19, trace_width 0.6, via_dia 0.6, via_drill 0.4
- rule pad_to_mask_clearance: 0.2 -> 0
- rule trace_clearance: 0.2 -> 0.19

Commit message: clean PCB DRC
Parts:
- C10, C11, C12, C13, C14, C5: footprint Capacitors_SMD:C_0805 -> Capacitors_SMD:C_0603
- moved J2 3.05 mm to (164.6, 50.0)
- moved P4 2.20 mm to (108.0, 45.2)
- moved P3 2.01 mm to (195.6, 45.4)
- moved R11 1.28 mm to (179.6, 56.0)
- moved J1 1.13 mm to (164.6, 54.0)
- moved J5 1.13 mm to (164.6, 52.0)
- moved C5 1.00 mm to (179.6, 53.2)
- moved P1 0.82 mm to (195.6, 32.0)
- moved R20 0.80 mm to (196.8, 73.4), turned to 0 degrees
- moved D6 0.20 mm to (196.8, 76.8)
- renumbered REF** to ?
Routing:
- net /SW_CTRL_PROT: track 0.00 -> 135.4 mm, vias 0 -> 4
- net /MCP_EVENT: track 0.00 -> 47.5 mm, vias 0 -> 4
- net /MCP_MCLR: track 0.00 -> 45.5 mm, vias 0 -> 6
- net Net-(R16-Pad2): track 0.00 -> 43.4 mm, vias 0 -> 2
- net Net-(R15-Pad2): track 0.00 -> 41.6 mm, vias 0 -> 2
- net Net-(L2-Pad2): track 0.00 -> 32.8 mm
- net Net-(C1-Pad1): track 0.00 -> 21.4 mm
- net Net-(D3-Pad1): track 0.00 -> 18.7 mm, vias 0 -> 2
- net Net-(C2-Pad2): track 0.00 -> 16.9 mm
- net +3V3: track 116.1 -> 129.3 mm, vias 2 -> 4
- net Net-(D1-Pad1): track 0.00 -> 10.6 mm, vias 0 -> 1
- net Net-(J2-Pad1): track 0.00 -> 10.4 mm
- net Net-(K2-Pad3): track 0.00 -> 10.2 mm
- net Net-(K2-Pad6): track 0.00 -> 9.95 mm
- net Net-(C3-Pad1): track 0.00 -> 9.52 mm
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