File: PowerMonitor.sch (KiCad schematic (older format))
At the start: 84 parts, among them J1 Conn_01x01, J10 TEST_1P, J11 TEST_1P, J12 TEST_1P, J13 TEST_1P, J14 TEST_1P, J15 TEST_1P, J16 Conn_01x03, J2 Conn_01x01, J3 Conn_01x01, J4 Conn_01x01, J5 Conn_01x01, J6 Conn_01x01, J7 Conn_01x01, J8 Conn_01x10, J9 TEST_1P, K1 T9AS5D12-5, K2 KEMET_UA2_5NJ, P1 Keystone_4912, P2 Keystone_4912, P3 Keystone_4912, P4 Keystone_4912, Q1 DMN3067LW, Q2 DMN3067LW, Q3 DMN3067LW, U1 IRM-02-5S, U2 IRM-05-5, U3 MCP39F521, U4 LP5907MFX-3.3, U5 ISO7731FDBQ, U6 ISO1540D

Commit message: layout started
Parts:
- added C15: 2.2uF 25V, Capacitors_SMD:C_0805, symbol C
- added J17: TEST_1P, nightmechanic_pcb:Keystone_50XX_TP, symbol TEST_1P
Connections:
- net +3.3V_ISO: now also C15.1
- net +5V: now also J17.1
- net GND: now also C15.2
- net Line_fused: now also R1.2; no longer L2.2
- net at C1.1, R5.1, U3.18 (V1-): now also L2.1; no longer R4.1
- new net: L2.2, R4.1
Other:
- moved on the sheet: J15, J16, J8, L2, R1, R3, R4
Changed lines of the file:
@@
 L R R1
 U 1 1 5AE27425
+P 2950 9600
+F 0 "R1" V 3030 9600 50  0000 C CNN
+F 1 "330k" V 2950 9600 50  0000 C CNN
+F 2 "Resistors_SMD:R_1206" V 2880 9600 50  0001 C CNN
+F 3 "" H 2950 9600 50  0001 C CNN
+	1    2950 9600
+	0    1    1    0
+$EndComp
+$Comp
+L R R3
+U 1 1 5AE276A4
 P 3550 9600
-F 0 "R1" V 3630 9600 50  0000 C CNN
+F 0 "R3" V 3630 9600 50  0000 C CNN
 F 1 "330k" V 3550 9600 50  0000 C CNN
 F 2 "Resistors_SMD:R_1206" V 3480 9600 50  0001 C CNN
@@
 $EndComp
 $Comp
-L R R3
-U 1 1 5AE276A4
+L R R4
+U 1 1 5AE27798
 P 4050 9600
-F 0 "R3" V 4130 9600 50  0000 C CNN
+F 0 "R4" V 4130 9600 50  0000 C CNN
 F 1 "330k" V 4050 9600 50  0000 C CNN
 F 2 "Resistors_SMD:R_1206" V 3980 9600 50  0001 C CNN
 F 3 "" H 4050 9600 50  0001 C CNN
 	1    4050 9600
-	0    1    1    0
-$EndComp
-$Comp
-L R R4
-U 1 1 5AE27798
-P 4500 9600
-F 0 "R4" V 4580 9600 50  0000 C CNN
-F 1 "330k" V 4500 9600 50  0000 C CNN
-F 2 "Resistors_SMD:R_1206" V 4430 9600 50  0001 C CNN
-F 3 "" H 4500 9600 50  0001 C CNN
-	1    4500 9600
 	0    1    1    0
 $EndComp
@@
 L Ferrite_Bead L2
 U 1 1 5AE28579
-P 2950 9600
-F 0 "L2" V 2800 9625 50  0000 C CNN
-F 1 "FB 300ohm" V 3100 9600 50  0000 C CNN
-F 2 "Capacitors_SMD:C_0805" V 2880 9600 50  0001 C CNN
-F 3 "" H 2950 9600 50  0001 C CNN
-	1    2950 9600
+P 4500 9600
+F 0 "L2" V 4350 9625 50  0000 C CNN
+F 1 "FB 300ohm" V 4650 9600 50  0000 C CNN
+F 2 "Capacitors_SMD:C_0805" V 4430 9600 50  0001 C CNN
+F 3 "" H 4500 9600 50  0001 C CNN
+	1    4500 9600
 	0    1    1    0
 $EndComp
@@
 L +5V #PWR011
 U 1 1 5AE9358C
-P 6400 2500
-F 0 "#PWR011" H 6400 2350 50  0001 C CNN
-F 1 "+5V" H 6400 2640 50  0000 C CNN
-F 2 "" H 6400 2500 50  0001 C CNN
-F 3 "" H 6400 2500 50  0001 C CNN
-	1    6400 2500
+P 6250 2500
+F 0 "#PWR011" H 6250 2350 50  0001 C CNN
+F 1 "+5V" H 6250 2640 50  0000 C CNN
+F 2 "" H 6250 2500 50  0001 C CNN
+F 3 "" H 6250 2500 50  0001 C CNN
+	1    6250 2500
 	1    0    0    -1
 $EndComp
@@
 L +5V_ISO #PWR035
 U 1 1 5AEA78C1
-P 15300 6150
-F 0 "#PWR035" H 15300 6000 50  0001 C CNN
-F 1 "+5V_ISO" H 15300 6290 50  0000 C CNN
-F 2 "" H 15300 6150 50  0001 C CNN
-F 3 "" H 15300 6150 50  0001 C CNN
-	1    15300 6150
+P 15450 6150
+F 0 "#PWR035" H 15450 6000 50  0001 C CNN
+F 1 "+5V_ISO" H 15450 6290 50  0000 C CNN
+F 2 "" H 15450 6150 50  0001 C CNN
+F 3 "" H 15450 6150 50  0001 C CNN
+	1    15450 6150
 	1    0    0    -1
 $EndComp
@@
 L GND_ISO #PWR036
 U 1 1 5AEA7B6E
-P 14800 6500
-F 0 "#PWR036" H 14800 6250 50  0001 C CNN
-F 1 "GND_ISO" H 14800 6350 50  0000 C CNN
-F 2 "" H 14800 6500 50  0001 C CNN
-F 3 "" H 14800 6500 50  0001 C CNN
-	1    14800 6500
+P 14950 6500
+F 0 "#PWR036" H 14950 6250 50  0001 C CNN
+F 1 "GND_ISO" H 14950 6350 50  0000 C CNN
+F 2 "" H 14950 6500 50  0001 C CNN
+F 3 "" H 14950 6500 50  0001 C CNN
+	1    14950 6500
 	1    0    0    -1
 $EndComp
@@
 L +3.3V_ISO #PWR037
 U 1 1 5AEA83C0
-P 15000 6400
-F 0 "#PWR037" H 15000 6250 50  0001 C CNN
-F 1 "+3.3V_ISO" H 15000 6540 50  0000 C CNN
-F 2 "" H 15000 6400 50  0001 C CNN
-F 3 "" H 15000 6400 50  0001 C CNN
-	1    15000 6400
+P 15150 6400
+F 0 "#PWR037" H 15150 6250 50  0001 C CNN
+F 1 "+3.3V_ISO" H 15150 6540 50  0000 C CNN
+F 2 "" H 15150 6400 50  0001 C CNN
+F 3 "" H 15150 6400 50  0001 C CNN
+	1    15150 6400
 	1    0    0    -1
 $EndComp
@@
 	1    0    0    -1
 $EndComp
-Text Label 15050 6700 0    60   ~ 0
+Text Label 15200 6700 0    60   ~ 0
 SDA_ISO
-Text Label 15050 6800 0    60   ~ 0
+Text Label 15200 6800 0    60   ~ 0
 SCL_ISO
-Text Label 14850 6900 0    60   ~ 0
+Text Label 15000 6900 0    60   ~ 0
 SW_CTRL_ISO
-Text Label 14850 7000 0    60   ~ 0
+Text Label 15000 7000 0    60   ~ 0
 MCLR_ISO
-Text Label 14850 7100 0    60   ~ 0
+Text Label 15000 7100 0    60   ~ 0
 EVENT_ISO
 $Comp
@@
 L PWR_FLAG #FLG043
 U 1 1 5AEABB56
-P 14650 6400
-F 0 "#FLG043" H 14650 6475 50  0001 C CNN
-F 1 "PWR_FLAG" H 14650 6550 50  0000 C CNN
-F 2 "" H 14650 6400 50  0001 C CNN
-F 3 "" H 14650 6400 50  0001 C CNN
-	1    14650 6400
+P 14800 6400
+F 0 "#FLG043" H 14800 6475 50  0001 C CNN
+F 1 "PWR_FLAG" H 14800 6550 50  0000 C CNN
+F 2 "" H 14800 6400 50  0001 C CNN
+F 3 "" H 14800 6400 50  0001 C CNN
+	1    14800 6400
 	1    0    0    -1
 $EndComp
@@
 L Conn_01x10 J8
 U 1 1 5AE8F11D
-P 15650 6700
-F 0 "J8" H 15650 7200 50  0000 C CNN
-F 1 "Conn_01x10" H 15650 6100 50  0000 C CNN
-F 2 "Pin_Headers:Pin_Header_Straight_1x10_Pitch2.54mm" H 15650 6700 50  0001 C CNN
-F 3 "" H 15650 6700 50  0001 C CNN
-	1    15650 6700
+P 15800 6700
+F 0 "J8" H 15800 7200 50  0000 C CNN
+F 1 "Conn_01x10" H 15800 6100 50  0000 C CNN
+F 2 "Pin_Headers:Pin_Header_Straight_1x10_Pitch2.54mm" H 15800 6700 50  0001 C CNN
+F 3 "" H 15800 6700 50  0001 C CNN
+	1    15800 6700
 	1    0    0    -1
 $EndComp
@@
 L GND_ISO #PWR050
 U 1 1 5AE8F345
-P 15250 7250
-F 0 "#PWR050" H 15250 7000 50  0001 C CNN
-F 1 "GND_ISO" H 15250 7100 50  0000 C CNN
-F 2 "" H 15250 7250 50  0001 C CNN
-F 3 "" H 15250 7250 50  0001 C CNN
-	1    15250 7250
+P 15400 7250
+F 0 "#PWR050" H 15400 7000 50  0001 C CNN
+F 1 "GND_ISO" H 15400 7100 50  0000 C CNN
+F 2 "" H 15400 7250 50  0001 C CNN
+F 3 "" H 15400 7250 50  0001 C CNN
+	1    15400 7250
 	1    0    0    -1
 $EndComp
@@
 L TEST_1P J15
 U 1 1 5AEB7626
-P 14250 6450
-F 0 "J15" H 14250 6720 50  0000 C CNN
-F 1 "TEST_1P" H 14250 6650 50  0000 C CNN
-F 2 "nightmechanic_pcb:Keystone_50XX_TP" H 14450 6450 50  0001 C CNN
-F 3 "" H 14450 6450 50  0001 C CNN
-	1    14250 6450
+P 14400 6450
+F 0 "J15" H 14400 6720 50  0000 C CNN
+F 1 "TEST_1P" H 14400 6650 50  0000 C CNN
+F 2 "nightmechanic_pcb:Keystone_50XX_TP" H 14600 6450 50  0001 C CNN
+F 3 "" H 14600 6450 50  0001 C CNN
+	1    14400 6450
 	1    0    0    -1
 $EndComp
@@
 L Conn_01x03 J16
 U 1 1 5AEBDA31
-P 14350 6800
-F 0 "J16" H 14350 7000 50  0000 C CNN
-F 1 "Conn_01x03" H 14350 6600 50  0000 C CNN
-F 2 "Pin_Headers:Pin_Header_Straight_1x03_Pitch2.54mm" H 14350 6800 50  0001 C CNN
-F 3 "" H 14350 6800 50  0001 C CNN
-	1    14350 6800
+P 14500 6800
+F 0 "J16" H 14500 7000 50  0000 C CNN
+F 1 "Conn_01x03" H 14500 6600 50  0000 C CNN
+F 2 "Pin_Headers:Pin_Header_Straight_1x03_Pitch2.54mm" H 14500 6800 50  0001 C CNN
+F 3 "" H 14500 6800 50  0001 C CNN
+	1    14500 6800
 	-1   0    0    -1
 $EndComp
@@
 L GND_ISO #PWR057
 U 1 1 5AEBE0E2
-P 14650 7000
-F 0 "#PWR057" H 14650 6750 50  0001 C CNN
-F 1 "GND_ISO" H 14650 6850 50  0000 C CNN
-F 2 "" H 14650 7000 50  0001 C CNN
-F 3 "" H 14650 7000 50  0001 C CNN
-	1    14650 7000
+P 14800 7000
+F 0 "#PWR057" H 14800 6750 50  0001 C CNN
+F 1 "GND_ISO" H 14800 6850 50  0000 C CNN
+F 2 "" H 14800 7000 50  0001 C CNN
+F 3 "" H 14800 7000 50  0001 C CNN
+	1    14800 7000
 	1    0    0    -1
 $EndComp
@@
 Wire Wire Line
 	6900 2550 8450 2550
-Wire Wire Line
-	7200 2550 7200 2650
 Connection ~ 7200 2550
 Wire Wire Line
@@
 	12500 2150 12500 9400
 Wire Wire Line
-	15300 6400 15450 6400
-Wire Wire Line
-	15300 6150 15300 6400
-Wire Wire Line
-	15450 6300 15300 6300
-Connection ~ 15300 6300
-Wire Wire Line
-	15000 6600 15450 6600
-Wire Wire Line
-	15000 6400 15000 6600
-Wire Wire Line
-	15450 6500 14800 6500
+	15450 6400 15600 6400
+Wire Wire Line
+	15450 6150 15450 6400
+Wire Wire Line
+	15600 6300 15450 6300
+Connection ~ 15450 6300
+Wire Wire Line
+	15150 6600 15600 6600
+Wire Wire Line
+	15150 6400 15150 6600
+Wire Wire Line
+	15600 6500 14950 6500
 Wire Wire Line
 	13200 7300 13200 6600
@@
 	13500 5950 13500 6100
 Wire Wire Line
-	14550 6700 15450 6700
-Wire Wire Line
-	14550 6800 15450 6800
-Wire Wire Line
-	14850 6900 15450 6900
-Wire Wire Line
-	14850 7000 15450 7000
-Wire Wire Line
-	14850 7100 15450 7100
+	14700 6700 15600 6700
+Wire Wire Line
+	14700 6800 15600 6800
+Wire Wire Line
+	15000 6900 15600 6900
+Wire Wire Line
+	15000 7000 15600 7000
+Wire Wire Line
+	15000 7100 15600 7100
 Wire Wire Line
 	9950 7750 9850 7750
@@
 	13900 8100 13900 8000
 Wire Wire Line
-	14250 6450 15000 6450
-Wire Wire Line
-	14650 6450 14650 6400
-Connection ~ 15000 6450
+	14000 6450 15150 6450
+Wire Wire Line
+	14800 6450 14800 6400
+Connection ~ 15150 6450
 Wire Wire Line
 	8650 1350 8650 1400
@@
 	7800 2500 7800 2550
 Connection ~ 7800 2550
-Wire Wire Line
-	6400 2500 6400 2550
-Connection ~ 6400 2550
 Wire Wire Line
 	3550 2900 3550 2950
@@
 Connection ~ 1500 2350
 Wire Wire Line
-	15450 7200 15250 7200
-Wire Wire Line
-	15250 7200 15250 7250
-Connection ~ 14650 6450
+	15600 7200 15400 7200
+Wire Wire Line
+	15400 7200 15400 7250
+Connection ~ 14800 6450
 Connection ~ 6500 5300
 Connection ~ 7700 4700
@@
 Connection ~ 14800 9150
 Wire Wire Line
-	14550 6900 14650 6900
-Wire Wire Line
-	14650 6900 14650 7000
+	14700 6900 14800 6900
+Wire Wire Line
+	14800 6900 14800 7000
 Wire Wire Line
 	3150 7900 1900 7900
@@
 Text Label 3950 1400 0    60   ~ 0
 Line_fused
+$Comp
+L C C15
+U 1 1 5AFCA661
+P 14000 6650
+F 0 "C15" H 14025 6750 50  0000 L CNN
+F 1 "2.2uF 25V" H 14025 6550 50  0000 L CNN
+F 2 "Capacitors_SMD:C_0805" H 14038 6500 50  0001 C CNN
+F 3 "" H 14000 6650 50  0001 C CNN
+	1    14000 6650
+	1    0    0    -1
+$EndComp
+Wire Wire Line
+	14000 6450 14000 6500
+Connection ~ 14400 6450
+Wire Wire Line
+	14000 6800 14000 6950
+$Comp
+L GND_ISO #PWR058
+U 1 1 5AFCB412
+P 14000 6950
+F 0 "#PWR058" H 14000 6700 50  0001 C CNN
+F 1 "GND_ISO" H 14000 6800 50  0000 C CNN
+F 2 "" H 14000 6950 50  0001 C CNN
+F 3 "" H 14000 6950 50  0001 C CNN
+	1    14000 6950
+	1    0    0    -1
+$EndComp
+$Comp
+L TEST_1P J17
+U 1 1 5AFCD1C1
+P 6500 2500
+F 0 "J17" H 6500 2770 50  0000 C CNN
+F 1 "TEST_1P" H 6500 2700 50  0000 C CNN
+F 2 "nightmechanic_pcb:Keystone_50XX_TP" H 6700 2500 50  0001 C CNN
+F 3 "" H 6700 2500 50  0001 C CNN
+	1    6500 2500
+	1    0    0    -1
+$EndComp
+Wire Wire Line
+	6250 2550 6250 2500
+Connection ~ 6250 2550
+Wire Wire Line
+	6500 2500 6500 2550
+Connection ~ 6500 2550
+Wire Wire Line
+	7200 2650 7200 2550
 $EndSCHEMATC

Commit message: clean PCB DRC
Parts:
- C10, C11, C12, C13, C14, C5: footprint Capacitors_SMD:C_0805 -> Capacitors_SMD:C_0603
Changed lines of the file:
@@
 F 0 "C5" H 6975 5650 50  0000 L CNN
 F 1 "0.1uF 25V" H 6975 5450 50  0000 L CNN
-F 2 "Capacitors_SMD:C_0805" H 6988 5400 50  0001 C CNN
+F 2 "Capacitors_SMD:C_0603" H 6988 5400 50  0001 C CNN
 F 3 "" H 6950 5550 50  0001 C CNN
 	1    6950 5550
@@
 F 0 "C10" H 9075 5650 50  0000 L CNN
 F 1 "0.1uF 25V" H 9075 5450 50  0000 L CNN
-F 2 "Capacitors_SMD:C_0805" H 9088 5400 50  0001 C CNN
+F 2 "Capacitors_SMD:C_0603" H 9088 5400 50  0001 C CNN
 F 3 "" H 9050 5550 50  0001 C CNN
 	1    9050 5550
@@
 F 0 "C11" H 11425 5150 50  0000 L CNN
 F 1 "0.1uF 25V" H 11425 4950 50  0000 L CNN
-F 2 "Capacitors_SMD:C_0805" H 11438 4900 50  0001 C CNN
+F 2 "Capacitors_SMD:C_0603" H 11438 4900 50  0001 C CNN
 F 3 "" H 11400 5050 50  0001 C CNN
 	1    11400 5050
@@
 F 0 "C13" H 13525 5050 50  0000 L CNN
 F 1 "0.1uF 25V" H 13525 4850 50  0000 L CNN
-F 2 "Capacitors_SMD:C_0805" H 13538 4800 50  0001 C CNN
+F 2 "Capacitors_SMD:C_0603" H 13538 4800 50  0001 C CNN
 F 3 "" H 13500 4950 50  0001 C CNN
 	1    13500 4950
@@
 F 0 "C12" H 11475 7000 50  0000 L CNN
 F 1 "0.1uF 25V" H 11475 6800 50  0000 L CNN
-F 2 "Capacitors_SMD:C_0805" H 11488 6750 50  0001 C CNN
+F 2 "Capacitors_SMD:C_0603" H 11488 6750 50  0001 C CNN
 F 3 "" H 11450 6900 50  0001 C CNN
 	1    11450 6900
@@
 F 0 "C14" H 13625 6950 50  0000 L CNN
 F 1 "0.1uF 25V" H 13625 6750 50  0000 L CNN
-F 2 "Capacitors_SMD:C_0805" H 13638 6700 50  0001 C CNN
+F 2 "Capacitors_SMD:C_0603" H 13638 6700 50  0001 C CNN
 F 3 "" H 13600 6850 50  0001 C CNN
 	1    13600 6850
